Commit message: [tiago/deburring] Move tags forwards, add parts to travelling_salesman.py script

File: urdf/P72-with-table.urdf (robot description, URDF)
Before this commit: robot p72, 48 links, 47 joints
Joints:
- joint to_tag_00001: origin xyz=0.160903806119 -0.0403379930677 0.593717015226 rpy=1.63558262861 0.003492408233 -0.0114843581192 -> xyz=0.160903806119 -0.0503379930677 0.593717015226 rpy=1.63558262861 0.003492408233 -0.0114843581192
- joint to_tag_00006: origin xyz=0.20594122137 -0.019883196378 0.270321366366 rpy=1.63559918028 -0.0219444636234 -0.0131355670517 -> xyz=0.20594122137 -0.029883196378 0.270321366366 rpy=1.63559918028 -0.0219444636234 -0.0131355670517
- joint to_tag_00015: origin xyz=-0.132714992453 -0.0338492746834 0.546713277339 rpy=1.63558443485 -0.0100636021863 -0.0123677826844 -> xyz=-0.132714992453 -0.0438492746834 0.546713277339 rpy=1.63558443485 -0.0100636021863 -0.0123677826844
- joint to_tag_00100: origin xyz=0.019355154887 -0.0352760613687 0.441859304771 rpy=1.66566275142 -0.00873291430813 0.0154183638448 -> xyz=0.019355154887 -0.0452760613687 0.441859304771 rpy=1.66566275142 -0.00873291430813 0.0154183638448
- joint to_tag_00101: origin xyz=0.0305993768382 -0.0495634897303 0.708105635544 rpy=1.60377606889 0.0126223907212 -0.00366126631718 -> xyz=0.0305993768382 -0.0595634897303 0.708105635544 rpy=1.60377606889 0.0126223907212 -0.00366126631718
